Commit message: Add 2D LiDAR sensor with Gazebo bridge and sensor world
- gpu_lidar in robot.xacro/robot.gazebo publishing /scan
- bridge /scan in bridge_parameters.yaml
- empty_with_sensors.sdf world; install worlds/ via CMakeLists
- update gazebo_model.launch.py and README; add resource.md notes
- ignore tf2 view_frames debug dumps

File: src/mobile_robot/model/robot.xacro (robot description, xacro)
@@ -1,4 +1,7 @@
 <?xml version="1.0"?>
 <robot name="differential_drive_robot" xmlns:xacro="http://www.ros.org/wiki/xacro">
+<!--______________________________________________________________________________________-->
+<!--_____________INERTIA AND BODY CONSTANTS_____________________________________________-->
+<!--______________________________________________________________________________________-->
 <!-- defining constants -->
 <xacro:property name="pi_const" value="3.14159265"/>
@@ -10,9 +13,12 @@
 <xacro:property name="r" value="0.15" />
 <xacro:property name="d" value="0.1" />
+<!--Lidar dimensions-->
+<xacro:property name="r_lidar" value="0.1" />
+<xacro:property name="d_lidar" value="0.1" />
 <xacro:property name="s1" value="${b/2+r}" />
 <xacro:property name="s2" value="${2*r}" />
 <xacro:property name="s3" value="${2*r}" />
 <xacro:property name="s4" value="${c/2+d/2}" />
- <!-- Mass Nd Inertial Properties-->
+<!-- Mass Nd Inertial Properties-->
 <!-- Body, Wheel, Caster Material Density-->
 <xacro:property name="d1" value="2710.0" />
@@ -56,11 +62,24 @@
     </inertial>
 </xacro:macro>
-<!-- For proper Robot control in Gazebo, we include some files-->
+<xacro:macro name="inertia_lidar">
+    <inertial>
+        <mass value="1e-6"/>
+        <origin xyz="0 0 0" rpy="0 0 0"/>
+        <inertia ixx="0.0001" ixy="0" ixz="0" iyy="0.0001" iyz="0" izz="0.0001"/>
+    </inertial>
+</xacro:macro>
+<!--______________________________________________________________________________________-->
+<!--_____________LINKS AND JOINTS_____________________________________________-->
+<!--______________________________________________________________________________________-->
+<!-- For proper Robot control in Gazebo, we include its gazebo file-->
 <xacro:include filename="$(find mobile_robot)/model/robot.gazebo" />
-<!-- Defining LINKS and JPINTS-->
 <link name="base_footprint" />  <!-- Fictious Link-->
+<!-- FUTURE ME: explicit origin prevents Physics.cc "world pose not available" crash loop.
+     Without this, dartsim tries to resolve lidar_link's world pose before
+     base_footprint->body_link is committed, causing entities 36/39 to loop. -->
 <joint name="body_link_joint" type="fixed">
     <parent link="base_footprint"/>
     <child link="body_link"/>
+    <origin xyz="0 0 0" rpy="0 0 0"/>
 </joint>
 <link name="body_link">
@@ -135,9 +154,4 @@
 </joint>
 <link name="caster_link">
-    <!-- <inertial>
-        <origin xyz="0.0 0.0 0.0" rpy="0.0 0.0 0.0"/>
-        <mass value="0.0"/>
-        <inertia ixx="0.0" ixy="0.0" ixz="0.0" iyy="0.0" iyz="0.0" izz="0.0"/>
-    </inertial> -->
     <visual name="">
         <origin xyz="0.0 0.0 0.0" rpy="0.0 0.0 0.0"/>
@@ -154,3 +168,33 @@
     <xacro:inertia_caster />
 </link>
+<!-- FUTURE ME: removed spurious <axis> tag — fixed joints have no rotation axis -->
+<!-- lidar_joint: placed on top of body_link surface.
+     body_link origin is at s1=b/2+r above base_footprint, and the box
+     half-height is b/2, so the top surface of the body is at s1+b/2 = b+r
+     above base_footprint. We place the lidar centre at that height + half
+     the lidar cylinder height so it sits neatly on top. -->
+<joint name="lidar_joint" type="fixed">
+    <parent link="body_link"/>
+    <child link="lidar_link"/>
+    <origin xyz="0 0 ${b+r+r_lidar/2}" rpy="0 0 0"/>
+</joint>
+<link name="lidar_link">
+    <!-- Visual and collision origins are 0 0 0 — the joint origin already
+         places the link centre correctly. Keeping offsets here caused the
+         sensor frame to be off-centre, tilting the scan plane. -->
+    <visual>
+        <origin xyz="0.0 0.0 0.0" rpy="0.0 0.0 0.0"/>
+        <geometry>
+            <cylinder radius="${r_lidar}" length="${d_lidar}"/>
+        </geometry>
+        <material name="Gazebo/Black"/>
+    </visual>
+    <collision>
+        <origin xyz="0.0 0.0 0.0" rpy="0.0 0.0 0.0"/>
+        <geometry>
+            <cylinder radius="${r_lidar}" length="${d_lidar}"/>
+        </geometry>
+    </collision>
+    <xacro:inertia_lidar />
+</link>
 </robot>

Commit message: migrated to ros2_control

File: src/mobile_robot/model/robot.xacro (robot description, xacro)
@@ -198,3 +198,27 @@
     <xacro:inertia_lidar />
 </link>
+<!--______________________________________________________________________________________-->
+<!--_____________CONTROL_____________________________________________-->
+<!--______________________________________________________________________________________-->
+<ros2_control name="GazeboSimSystem" type="system">
+        <hardware>
+            <plugin>gz_ros2_control/GazeboSimSystem</plugin>
+        </hardware>
+        <joint name="wheel1_joint">
+            <command_interface name="velocity">
+                <param name="min">-10</param>
+                <param name="max">10</param>
+            </command_interface>
+            <state_interface name="velocity"></state_interface>
+            <state_interface name="position"></state_interface>
+        </joint>
+        <joint name="wheel2_joint">
+            <command_interface name="velocity">
+                <param name="min">-10</param>
+                <param name="max">10</param>
+            </command_interface>
+            <state_interface name="velocity"></state_interface>
+            <state_interface name="position"></state_interface>
+         </joint>
+    </ros2_control>
 </robot>

Commit message: SLAM integrated, bug fixes

File: src/mobile_robot/model/robot.xacro (robot description, xacro)
@@ -81,5 +81,5 @@
     <parent link="base_footprint"/>
     <child link="body_link"/>
-    <origin xyz="0 0 0" rpy="0 0 0"/>
+    <origin xyz="${s2} 0 0" rpy="0 0 0"/>
 </joint>
 <link name="body_link">

Commit message: camera + OpenCV obstacle detection feeding local costmap; footprint polygon
- rgbd_camera sensor, camera_link + camera_link_optical, image/points/camera_info bridged
- camera_opencv.py: HSV threshold -> filtered PointCloud2 on /detected_obstacle_points
- local costmap voxel_layer consumes the cloud; global costmap stays scan-only
- robot_radius -> footprint polygon (base_footprint sits 0.3 m behind chassis centre)
- MPPI consider_footprint enabled; trajectory_point_step 2->4 to hold 20 Hz

Verified against a 0.32 m coffee table that sits below the lidar plane and is
therefore absent from both /scan and the saved map: detector off, the rover
drives through it; detector on, it stops short and routes around.

Known limit: a single forward camera observes only an obstacle's near face, so
the marked region is thinner than the real object.

File: src/mobile_robot/model/robot.xacro (robot description, xacro)
@@ -16,4 +16,6 @@
 <xacro:property name="r_lidar" value="0.1" />
 <xacro:property name="d_lidar" value="0.1" />
+<xacro:property name="r_camera" value="0.025" />
+<xacro:property name="d_camera" value="0.025" />
 <xacro:property name="s1" value="${b/2+r}" />
 <xacro:property name="s2" value="${2*r}" />
@@ -69,4 +71,11 @@
     </inertial>
 </xacro:macro>
+<xacro:macro name="inertia_camera">
+    <inertial>
+        <mass value="1e-6"/>
+        <origin xyz="0 0 0" rpy="0 0 0"/>
+        <inertia ixx="0.0001" ixy="0" ixz="0" iyy="0.0001" iyz="0" izz="0.0001"/>
+    </inertial>
+</xacro:macro>
 <!--______________________________________________________________________________________-->
 <!--_____________LINKS AND JOINTS_____________________________________________-->
@@ -198,4 +207,25 @@
     <xacro:inertia_lidar />
 </link>
+<joint name="camera_joint" type="fixed">
+    <parent link="body_link"/>
+    <child link="camera_link"/>
+    <origin xyz="0.505 0 ${s1}" rpy="0 0 0"/>
+</joint>
+<link name="camera_link">
+    <visual>
+        <origin xyz="0.0 0.0 0.0" rpy="0.0 0.0 0.0"/>
+        <geometry>
+            <box size="0.010 0.03 0.03"/>
+        </geometry>
+        <material name="Gazebo/Black"/>
+    </visual>
+    <xacro:inertia_camera/>
+</link>
+<joint name="camera_optical_joint" type="fixed">
+    <parent link="camera_link"/>
+    <child link="camera_link_optical"/>
+    <origin xyz="0 0 0" rpy="${-pi_const/2} 0.0 ${-pi_const/2}"/>
+</joint>
+<link name="camera_link_optical"></link>
 <!--______________________________________________________________________________________-->
 <!--_____________CONTROL_____________________________________________-->
